File: hardware/pcb/xim.kicad_sch (KiCad schematic)
At the start: 72 parts, among them IC1 RP2040_QFN56, SW1 RKB2, SW2 RKB2, U1 8MB QSPI, U2 RT9080-3.3, U3 SY6280AAC, U4 FE1.1s, X2 USB A, X3 USB A, X6 USB Type C, X7 USB Type C, Y1 12MHz/12pF, Y2 12MHz/20pF

Commit message: feat(hardware): add SWD test pads
Parts:
- added TP4: SWCLK, Adafruit Feather RP2040 USB Host-import-fps:TESTPOINT_ROUND_1.5MM_NO, symbol Adafruit Feather RP2040 USB Host-eagle-import:TESTPOINTROUND1.5MMNO
- added TP5: SWDIO, Adafruit Feather RP2040 USB Host-import-fps:TESTPOINT_ROUND_1.5MM_NO, symbol Adafruit Feather RP2040 USB Host-eagle-import:TESTPOINTROUND1.5MMNO
- added TP6: GND, Adafruit Feather RP2040 USB Host-import-fps:TESTPOINT_ROUND_1.5MM_NO, symbol Adafruit Feather RP2040 USB Host-eagle-import:TESTPOINTROUND1.5MMNO
Connections:
- net GND: now also TP6.P$1
- net SWCLK: now reaches IC1.24 (SWCLK)
- net SWCLK: now also TP4.P$1
- net SWDIO: now reaches IC1.25 (SWDIO)
- net SWDIO: now also TP5.P$1
- no-connect marks 39 -> 37
